Commit message: g

File: src/ned-ros2-driver/niryo_ned_description/urdf/tools/niryo_gripper1.urdf.xacro (robot description, xacro)
@@ -1,6 +1,7 @@
 <?xml version="1.0"?>
 <robot xmlns:xacro="http://www.ros.org/wiki/xacro" name="niryo_ned2">
+    <xacro:macro name="gripper_1" params="prefix">
     <!-- Base Gripper -->
-    <link name="base_gripper_1">
+    <link name="${prefix}base_gripper_1">
         <inertial>
             <origin xyz="0.0028582 0.0022204 0.023772"
@@ -34,5 +35,5 @@
     <!-- Mors 1 -->
     <link
-            name="mors_1">
+            name="${prefix}mors_1">
         <inertial>
             <origin xyz="-0.0049739 0.0067393 -0.023929"
@@ -68,10 +69,10 @@
     </link>
     <joint
-            name="joint_base_to_mors_1"
+            name="${prefix}joint_base_to_mors_1"
             type="prismatic">
         <origin xyz="0.01455 -0.0796 0.0096137"
                 rpy="1.5708 0 0"/>
-        <parent link="base_gripper_1"/>
-        <child link="mors_1"/>
+        <parent link="${prefix}base_gripper_1"/>
+        <child link="${prefix}mors_1"/>
         <axis xyz="0 1 0"/>
         <limit lower="-0.01"
@@ -82,5 +83,5 @@
     <!-- Mors 2 -->
     <link
-            name="mors_2">
+            name="${prefix}mors_2">
         <inertial>
             <origin xyz="-0.0049739 -0.0067393 -0.023929"
@@ -112,10 +113,10 @@
         </collision>
     </link>
-    <joint name="joint_base_to_mors_2"
+    <joint name="${prefix}joint_base_to_mors_2"
            type="prismatic">
         <origin xyz="0.01455 -0.0796 -0.011066"
                 rpy="1.5708 0 0"/>
-        <parent link="base_gripper_1"/>
-        <child link="mors_2"/>
+        <parent link="${prefix}base_gripper_1"/>
+        <child link="${prefix}mors_2"/>
         <axis xyz="0 -1 0"/>
         <limit lower="-0.01"
@@ -124,3 +125,4 @@
                velocity="5"/>
     </joint>
+    </xacro:macro>
 </robot>
